File: CIRCUITOS/alimentacion.kicad_sch (KiCad schematic)
At the start: 0 parts

Commit message: Agregue TP11
Parts:
- added C1: C, symbol Device:C
- added D5: D, symbol Device:D
- added J1, J2: Conn_01x02_Pin, symbol Connector:Conn_01x02_Pin
- added U7: L7805, symbol Regulator_Linear:L7805
