File: CIRCUITOS/monitoreo_termico.kicad_sch (KiCad schematic)
At the start: 0 parts

Commit message: Agregue TP11
Parts:
- added R1, R4: 10K, symbol Device:R
- added R2: 5K, symbol Device:R_Variable
- added R3: 40K, symbol Device:R
- added R5: 5K, symbol Device:R
- added R6: 200K, symbol Device:R_Variable
- added U1, U2, U4: LM358, symbol Amplifier_Operational:LM358
- added U3: LM35-D, Package_SO:SOIC-8_3.9x4.9mm_P1.27mm, symbol Sensor_Temperature:LM35-D
Connections:
- new net: R6.2, U4.1
- new net: R5.2, R6.1, U4.2 (-)
- new net: R3.1, U1.1, U4.3 (+)
- new net: U1.3 (+), U2.1, U2.2 (-)
- new net: U2.3 (+), U3.1 (V_{OUT})
- new net: R3.2, R4.1, U1.2 (-)
- new net: R1.2, R2.1, R5.1
- new net +9V: R1.1, U3.8 (+V_{S})
- new net GND: R2.2, R4.2, U3.4 (GND)
Other:
- note added: "Vref"
